File: ADC.sch (KiCad schematic (older format))
At the start: 0 parts

Commit message: First release of the schematic.
Parts:
- added C58, C60: 0.1uF, symbol C_Small
- added C59: 47uF, symbol C_Small
- added C61: 10uF, symbol C_Small
- added C62: 390pF, symbol C_Small
- added C63: 5600pF, symbol C_Small
- added J5: TEST_1P, symbol TEST_1P
- added R36, R37: 10k, symbol R
- added R38: 560, symbol R
- added U11: AD1939WBSTZ, symbol AD1939WBSTZ
- added U12: 74LVC1G08, symbol 74LVC1G08
- added U13: FOX924B - 12.288MHz, symbol FOX924B
Connections:
- net labels added: +3.3V, +3.3VA, ABCLK, ADC1LN, ADC1LP, ADC1RN, ADC1RP, ADC2LN, ADC2LP, ADC2RN, ADC2RP, ALRCLK, ASDATA1, ASDATA2, GNDA, GNDD, SPI_CLK, SPI_MISO, SPI_MOSI, ~AD1939_CS, ~AD1939_SOFT_RESET, ~RESET
- wire segments 0 -> 50
- no-connect marks 0 -> 27

Commit message: First schematic release
Parts:
- C58, C60, C61, C62, C63: footprint (none) -> Capacitors_SMD:C_0603_HandSoldering
- C59: footprint (none) -> Capacitors_SMD:C_1206_HandSoldering
- J5: footprint (none) -> SMD_Packages:1Pin
- R36, R37, R38: footprint (none) -> Resistors_SMD:R_0603_HandSoldering
- U11: footprint (none) -> Housings_QFP:LQFP-64_10x10mm_Pitch0.5mm
- U12: footprint (none) -> TO_SOT_Packages_SMD:SOT-353
- U13: footprint (none) -> Zeabus:Oscillator-TCXO
Changed lines of the file:
@@
 LIBS:zeabus
 LIBS:ftdi
+LIBS:Zeabus-Elec-Hydrophone-cache
 EELAYER 25 0
 EELAYER END
@@
 F 0 "U11" H 6114 1959 45  0000 L BNN
 F 1 "AD1939WBSTZ" H 6077 1859 45  0000 L BNN
-F 2 "" H 4830 1750 20  0001 C CNN
+F 2 "Housings_QFP:LQFP-64_10x10mm_Pitch0.5mm" H 4830 1750 20  0001 C CNN
 F 3 "" H 4800 1600 60  0001 C CNN
 	1    4800 1600
@@
 F 0 "U13" H 8500 3850 45  0000 L BNN
 F 1 "FOX924B - 12.288MHz" H 7900 3100 45  0000 L BNN
-F 2 "" H 8980 3350 20  0001 C CNN
+F 2 "Zeabus:Oscillator-TCXO" H 8980 3350 20  0001 C CNN
 F 3 "" H 8950 3200 60  0001 C CNN
 	1    8950 3200
@@
 NoConn ~ 10150 2700
 $Comp
-L GNDD #PWR065
+L GNDD #PWR066
 U 1 1 59966FCA
 P 10150 3100
-F 0 "#PWR065" H 10150 2850 50  0001 C CNN
+F 0 "#PWR066" H 10150 2850 50  0001 C CNN
 F 1 "GNDD" H 10150 2950 50  0000 C CNN
 F 2 "" H 10150 3100 50  0001 C CNN
@@
 $EndComp
 $Comp
-L GNDA #PWR066
+L GNDA #PWR067
 U 1 1 5996700C
 P 8150 2600
-F 0 "#PWR066" H 8150 2350 50  0001 C CNN
+F 0 "#PWR067" H 8150 2350 50  0001 C CNN
 F 1 "GNDA" H 8150 2450 50  0000 C CNN
 F 2 "" H 8150 2600 50  0001 C CNN
@@
 $EndComp
 $Comp
-L +3.3V #PWR067
+L +3.3V #PWR068
 U 1 1 59967026
 P 9050 2700
-F 0 "#PWR067" H 9050 2550 50  0001 C CNN
+F 0 "#PWR068" H 9050 2550 50  0001 C CNN
 F 1 "+3.3V" H 9050 2840 50  0000 C CNN
 F 2 "" H 9050 2700 50  0001 C CNN
@@
 $EndComp
 $Comp
-L +3.3VA #PWR068
+L +3.3VA #PWR069
 U 1 1 59967068
 P 4800 1400
-F 0 "#PWR068" H 4800 1250 50  0001 C CNN
+F 0 "#PWR069" H 4800 1250 50  0001 C CNN
 F 1 "+3.3VA" H 4800 1540 50  0000 C CNN
 F 2 "" H 4800 1400 50  0001 C CNN
@@
 F 0 "J5" H 8500 3270 50  0000 C CNN
 F 1 "TEST_1P" H 8500 3200 50  0000 C CNN
-F 2 "" H 8700 3000 50  0001 C CNN
+F 2 "SMD_Packages:1Pin" H 8700 3000 50  0001 C CNN
 F 3 "" H 8700 3000 50  0001 C CNN
 	1    8500 3000
@@
 $EndComp
 $Comp
-L GNDD #PWR069
+L GNDD #PWR070
 U 1 1 599671EA
 P 8150 2200
-F 0 "#PWR069" H 8150 1950 50  0001 C CNN
+F 0 "#PWR070" H 8150 1950 50  0001 C CNN
 F 1 "GNDD" H 8150 2050 50  0000 C CNN
 F 2 "" H 8150 2200 50  0001 C CNN
@@
 	7800 3800 8200 3800
 $Comp
-L +3.3V #PWR070
+L +3.3V #PWR071
 U 1 1 59967361
 P 4500 2100
-F 0 "#PWR070" H 4500 1950 50  0001 C CNN
+F 0 "#PWR071" H 4500 1950 50  0001 C CNN
 F 1 "+3.3V" H 4500 2240 50  0000 C CNN
 F 2 "" H 4500 2100 50  0001 C CNN
@@
 	4500 3000 4800 3000
 $Comp
-L GNDD #PWR071
+L GNDD #PWR072
 U 1 1 59967561
 P 4500 3300
-F 0 "#PWR071" H 4500 3050 50  0001 C CNN
+F 0 "#PWR072" H 4500 3050 50  0001 C CNN
 F 1 "GNDD" H 4500 3150 50  0000 C CNN
 F 2 "" H 4500 3300 50  0001 C CNN
@@
 F 0 "U12" H 3050 4050 50  0000 C CNN
 F 1 "74LVC1G08" H 3050 3950 50  0000 C CNN
-F 2 "" H 3050 4000 50  0001 C CNN
+F 2 "TO_SOT_Packages_SMD:SOT-353" H 3050 4000 50  0001 C CNN
 F 3 "" H 3050 4000 50  0001 C CNN
 	1    3050 4000
@@
 $EndComp
 $Comp
-L GNDD #PWR072
+L GNDD #PWR073
 U 1 1 599681C6
 P 2900 4300
-F 0 "#PWR072" H 2900 4050 50  0001 C CNN
+F 0 "#PWR073" H 2900 4050 50  0001 C CNN
 F 1 "GNDD" H 2900 4150 50  0000 C CNN
 F 2 "" H 2900 4300 50  0001 C CNN
@@
 $EndComp
 $Comp
-L +3.3V #PWR073
+L +3.3V #PWR074
 U 1 1 599681FD
 P 2900 3700
-F 0 "#PWR073" H 2900 3550 50  0001 C CNN
+F 0 "#PWR074" H 2900 3550 50  0001 C CNN
 F 1 "+3.3V" H 2900 3840 50  0000 C CNN
 F 2 "" H 2900 3700 50  0001 C CNN
@@
 F 0 "C58" H 2760 5270 50  0000 L CNN
 F 1 "0.1uF" H 2760 5120 50  0000 L CNN
-F 2 "" H 2750 5200 50  0001 C CNN
+F 2 "Capacitors_SMD:C_0603_HandSoldering" H 2750 5200 50  0001 C CNN
 F 3 "" H 2750 5200 50  0001 C CNN
 	1    2750 5200
@@
 F 0 "C59" H 3060 5270 50  0000 L CNN
 F 1 "47uF" H 3060 5120 50  0000 L CNN
-F 2 "" H 3050 5200 50  0001 C CNN
+F 2 "Capacitors_SMD:C_1206_HandSoldering" H 3050 5200 50  0001 C CNN
 F 3 "" H 3050 5200 50  0001 C CNN
 	1    3050 5200
@@
 F 0 "C60" H 3460 5270 50  0000 L CNN
 F 1 "0.1uF" H 3460 5120 50  0000 L CNN
-F 2 "" H 3450 5200 50  0001 C CNN
+F 2 "Capacitors_SMD:C_0603_HandSoldering" H 3450 5200 50  0001 C CNN
 F 3 "" H 3450 5200 50  0001 C CNN
 	1    3450 5200
@@
 F 0 "C61" H 3710 5270 50  0000 L CNN
 F 1 "10uF" H 3710 5120 50  0000 L CNN
-F 2 "" H 3700 5200 50  0001 C CNN
+F 2 "Capacitors_SMD:C_0603_HandSoldering" H 3700 5200 50  0001 C CNN
 F 3 "" H 3700 5200 50  0001 C CNN
 	1    3700 5200
@@
 F 0 "R36" V 2430 3600 50  0000 C CNN
 F 1 "10k" V 2350 3600 50  0000 C CNN
-F 2 "" V 2280 3600 50  0001 C CNN
+F 2 "Resistors_SMD:R_0603_HandSoldering" V 2280 3600 50  0001 C CNN
 F 3 "" H 2350 3600 50  0001 C CNN
 	1    2350 3600
@@
 F 0 "R37" V 2530 5250 50  0000 C CNN
 F 1 "10k" V 2450 5250 50  0000 C CNN
-F 2 "" V 2380 5250 50  0001 C CNN
+F 2 "Resistors_SMD:R_0603_HandSoldering" V 2380 5250 50  0001 C CNN
 F 3 "" H 2450 5250 50  0001 C CNN
 	1    2450 5250
@@
 $EndComp
 $Comp
-L GNDD #PWR074
+L GNDD #PWR075
 U 1 1 59968BAE
 P 3050 5350
-F 0 "#PWR074" H 3050 5100 50  0001 C CNN
+F 0 "#PWR075" H 3050 5100 50  0001 C CNN
 F 1 "GNDD" H 3050 5200 50  0000 C CNN
 F 2 "" H 3050 5350 50  0001 C CNN
@@
 Connection ~ 2350 3900
 $Comp
-L +3.3V #PWR075
+L +3.3V #PWR076
 U 1 1 59968D2B
 P 2350 3450
-F 0 "#PWR075" H 2350 3300 50  0001 C CNN
+F 0 "#PWR076" H 2350 3300 50  0001 C CNN
 F 1 "+3.3V" H 2350 3590 50  0000 C CNN
 F 2 "" H 2350 3450 50  0001 C CNN
@@
 $EndComp
 $Comp
-L +3.3V #PWR076
+L +3.3V #PWR077
 U 1 1 59968D54
 P 2450 5100
-F 0 "#PWR076" H 2450 4950 50  0001 C CNN
+F 0 "#PWR077" H 2450 4950 50  0001 C CNN
 F 1 "+3.3V" H 2450 5240 50  0000 C CNN
 F 2 "" H 2450 5100 50  0001 C CNN
@@
 F 0 "C62" H 4160 6120 50  0000 L CNN
 F 1 "390pF" H 4160 5970 50  0000 L CNN
-F 2 "" H 4150 6050 50  0001 C CNN
+F 2 "Capacitors_SMD:C_0603_HandSoldering" H 4150 6050 50  0001 C CNN
 F 3 "" H 4150 6050 50  0001 C CNN
 	1    4150 6050
@@
 F 0 "C63" H 4410 6420 50  0000 L CNN
 F 1 "5600pF" H 4410 6270 50  0000 L CNN
-F 2 "" H 4400 6350 50  0001 C CNN
+F 2 "Capacitors_SMD:C_0603_HandSoldering" H 4400 6350 50  0001 C CNN
 F 3 "" H 4400 6350 50  0001 C CNN
 	1    4400 6350
@@
 F 0 "R38" V 4030 6350 50  0000 C CNN
 F 1 "560" V 3950 6350 50  0000 C CNN
-F 2 "" V 3880 6350 50  0001 C CNN
+F 2 "Resistors_SMD:R_0603_HandSoldering" V 3880 6350 50  0001 C CNN
 F 3 "" H 3950 6350 50  0001 C CNN
 	1    3950 6350
@@
 Connection ~ 4800 6050
 $Comp
-L +3.3VA #PWR077
+L +3.3VA #PWR078
 U 1 1 599691FE
 P 3800 6050
-F 0 "#PWR077" H 3800 5900 50  0001 C CNN
+F 0 "#PWR078" H 3800 5900 50  0001 C CNN
 F 1 "+3.3VA" H 3800 6190 50  0000 C CNN
 F 2 "" H 3800 6050 50  0001 C CNN

Commit message: - Add C150 - C153 at LNA input - Change value of C112, C115, C118, C221 at LNA input - Finished PCB lay-out. Ready to route
Parts:
- C58, C60, C61, C62, C63: footprint Capacitors_SMD:C_0603_HandSoldering -> Capacitors_SMD:C_0603
- C59: footprint Capacitors_SMD:C_1206_HandSoldering -> Capacitors_SMD:C_0603
- J5: footprint SMD_Packages:1Pin -> Zeabus:1Pin-TP
- R36, R37, R38: footprint Resistors_SMD:R_0603_HandSoldering -> Resistors_SMD:R_0603
Changed lines of the file:
@@
 F 0 "J5" H 8500 3270 50  0000 C CNN
 F 1 "TEST_1P" H 8500 3200 50  0000 C CNN
-F 2 "SMD_Packages:1Pin" H 8700 3000 50  0001 C CNN
+F 2 "Zeabus:1Pin-TP" H 8700 3000 50  0001 C CNN
 F 3 "" H 8700 3000 50  0001 C CNN
 	1    8500 3000
@@
 F 0 "C58" H 2760 5270 50  0000 L CNN
 F 1 "0.1uF" H 2760 5120 50  0000 L CNN
-F 2 "Capacitors_SMD:C_0603_HandSoldering" H 2750 5200 50  0001 C CNN
+F 2 "Capacitors_SMD:C_0603" H 2750 5200 50  0001 C CNN
 F 3 "" H 2750 5200 50  0001 C CNN
 	1    2750 5200
@@
 F 0 "C59" H 3060 5270 50  0000 L CNN
 F 1 "47uF" H 3060 5120 50  0000 L CNN
-F 2 "Capacitors_SMD:C_1206_HandSoldering" H 3050 5200 50  0001 C CNN
+F 2 "Capacitors_SMD:C_0603" H 3050 5200 50  0001 C CNN
 F 3 "" H 3050 5200 50  0001 C CNN
 	1    3050 5200
@@
 F 0 "C60" H 3460 5270 50  0000 L CNN
 F 1 "0.1uF" H 3460 5120 50  0000 L CNN
-F 2 "Capacitors_SMD:C_0603_HandSoldering" H 3450 5200 50  0001 C CNN
+F 2 "Capacitors_SMD:C_0603" H 3450 5200 50  0001 C CNN
 F 3 "" H 3450 5200 50  0001 C CNN
 	1    3450 5200
@@
 F 0 "C61" H 3710 5270 50  0000 L CNN
 F 1 "10uF" H 3710 5120 50  0000 L CNN
-F 2 "Capacitors_SMD:C_0603_HandSoldering" H 3700 5200 50  0001 C CNN
+F 2 "Capacitors_SMD:C_0603" H 3700 5200 50  0001 C CNN
 F 3 "" H 3700 5200 50  0001 C CNN
 	1    3700 5200
@@
 F 0 "R36" V 2430 3600 50  0000 C CNN
 F 1 "10k" V 2350 3600 50  0000 C CNN
-F 2 "Resistors_SMD:R_0603_HandSoldering" V 2280 3600 50  0001 C CNN
+F 2 "Resistors_SMD:R_0603" V 2280 3600 50  0001 C CNN
 F 3 "" H 2350 3600 50  0001 C CNN
 	1    2350 3600
@@
 F 0 "R37" V 2530 5250 50  0000 C CNN
 F 1 "10k" V 2450 5250 50  0000 C CNN
-F 2 "Resistors_SMD:R_0603_HandSoldering" V 2380 5250 50  0001 C CNN
+F 2 "Resistors_SMD:R_0603" V 2380 5250 50  0001 C CNN
 F 3 "" H 2450 5250 50  0001 C CNN
 	1    2450 5250
@@
 F 0 "C62" H 4160 6120 50  0000 L CNN
 F 1 "390pF" H 4160 5970 50  0000 L CNN
-F 2 "Capacitors_SMD:C_0603_HandSoldering" H 4150 6050 50  0001 C CNN
+F 2 "Capacitors_SMD:C_0603" H 4150 6050 50  0001 C CNN
 F 3 "" H 4150 6050 50  0001 C CNN
 	1    4150 6050
@@
 F 0 "C63" H 4410 6420 50  0000 L CNN
 F 1 "5600pF" H 4410 6270 50  0000 L CNN
-F 2 "Capacitors_SMD:C_0603_HandSoldering" H 4400 6350 50  0001 C CNN
+F 2 "Capacitors_SMD:C_0603" H 4400 6350 50  0001 C CNN
 F 3 "" H 4400 6350 50  0001 C CNN
 	1    4400 6350
@@
 F 0 "R38" V 4030 6350 50  0000 C CNN
 F 1 "560" V 3950 6350 50  0000 C CNN
-F 2 "Resistors_SMD:R_0603_HandSoldering" V 3880 6350 50  0001 C CNN
+F 2 "Resistors_SMD:R_0603" V 3880 6350 50  0001 C CNN
 F 3 "" H 3950 6350 50  0001 C CNN
 	1    3950 6350
