File: DSP-External_Port.sch (KiCad schematic (older format))
At the start: 62 parts, among them J1 JTAG, SW1 SW_DIP_x02, U1 ADSP-21489BSWZ-4B, U2 FOX924B - 25MHz

Commit message: First schematic release
Parts:
- C1, C10, C11, C12, C13, C14, C15, C16, C17, C18, C19, C2, C20, C21, C22, C23, C24, C25, C26, C27, C28, C29, C3, C30, C31, C32, C33, C34, C35, C36, C37, C38, C39, C4, C40, C41, C42, C43, C44, C5, C6, C7, C8, C9: footprint (none) -> Capacitors_SMD:C_0603_HandSoldering
- J1: footprint (none) -> Pin_Headers:Pin_Header_Straight_2x07_Pitch2.54mm
- R1, R2, R3, R4, R5, R6, R7, R8, R9: footprint (none) -> Resistors_SMD:R_0603_HandSoldering
- RN1, RN2, RN3, RN4, RN5: footprint (none) -> Zeabus:CRA06S
- SW1: footprint (none) -> Buttons_Switches_SMD:SW_DIP_x2_W5.08mm_Slide_Copal_CHS-A
- U1: footprint (none) -> Zeabus:ADSP-21489-177
- U2: footprint (none) -> Zeabus:Oscillator-TCXO

Commit message: - Add C150 - C153 at LNA input - Change value of C112, C115, C118, C221 at LNA input - Finished PCB lay-out. Ready to route
Parts:
- C1, C10, C11, C12, C13, C14, C15, C16, C17, C18, C19, C2, C20, C21, C22, C23, C24, C25, C26, C27, C28, C29, C3, C30, C31, C32, C33, C34, C35, C36, C37, C38, C39, C4, C40, C41, C42, C43, C44, C5, C6, C7, C8, C9: footprint Capacitors_SMD:C_0603_HandSoldering -> Capacitors_SMD:C_0603
- R1, R2, R3, R4, R5, R6, R7, R8, R9: footprint Resistors_SMD:R_0603_HandSoldering -> Resistors_SMD:R_0603
