File: DSP-Memory.sch (KiCad schematic (older format))
At the start: 32 parts, among them J22 TEST_1P, SW2 SW_Push_Dual, U1 ADSP-21489BSWZ-4B, U3 S29GL032N, U4 74LVC1G08, U5 74LVC1G08, U6 ADM708SARZ, Y1 CSTCC2M00G53-R0

Commit message: First schematic release
Parts:
- C45, C46, C47, JP1: footprint (none) -> Capacitors_SMD:C_0603_HandSoldering
- D1: footprint (none) -> LEDs:LED_0603
- J22: footprint (none) -> SMD_Packages:1Pin
- JP2: footprint (none) -> Pin_Headers:Pin_Header_Straight_1x02_Pitch2.54mm
- R10, R11, R12, R13, R14, R15, R16, R17, R18, R19: footprint (none) -> Resistors_SMD:R_0603_HandSoldering
- RN10, RN11, RN12, RN13, RN6, RN7, RN8, RN9: footprint (none) -> Zeabus:CRA06S
- SW2: value SW_Push_Dual -> PB; footprint (none) -> Zeabus:Button-EVQ
- U1: footprint (none) -> Zeabus:ADSP-21489-177
- U3: footprint (none) -> Housings_SSOP:TSOP-I-48_12x18.4mm_Pitch0.5mm
- U4, U5: footprint (none) -> TO_SOT_Packages_SMD:SOT-353
- U6: footprint (none) -> Zeabus:ADM708_R_8
- Y1: footprint (none) -> Crystals:Resonator_7.2x3mm
Changed lines of the file:
@@
 LIBS:zeabus
 LIBS:ftdi
+LIBS:Zeabus-Elec-Hydrophone-cache
 EELAYER 25 0
 EELAYER END
@@
 F 0 "U1" H 4700 4300 45  0000 L BNN
 F 1 "ADSP-21489BSWZ-4B" H 4700 1000 45  0000 L BNN
-F 2 "" H 5430 2750 20  0001 C CNN
+F 2 "Zeabus:ADSP-21489-177" H 5430 2750 20  0001 C CNN
 F 3 "" H 5400 2600 60  0001 C CNN
 	1    5400 2600
@@
 F 0 "U3" H 8650 1500 60  0000 C CNN
 F 1 "S29GL032N" H 8850 -1200 60  0000 C CNN
-F 2 "" H 8350 1400 60  0001 C CNN
+F 2 "Housings_SSOP:TSOP-I-48_12x18.4mm_Pitch0.5mm" H 8350 1400 60  0001 C CNN
 F 3 "" H 8350 1400 60  0001 C CNN
 	1    8350 1400
@@
 F 0 "R14" V 7680 3350 50  0000 C CNN
 F 1 "10k" V 7600 3350 50  0000 C CNN
-F 2 "" V 7530 3350 50  0001 C CNN
+F 2 "Resistors_SMD:R_0603_HandSoldering" V 7530 3350 50  0001 C CNN
 F 3 "" H 7600 3350 50  0001 C CNN
 	1    7600 3350
@@
 F 0 "R13" V 7480 3350 50  0000 C CNN
 F 1 "10k" V 7400 3350 50  0000 C CNN
-F 2 "" V 7330 3350 50  0001 C CNN
+F 2 "Resistors_SMD:R_0603_HandSoldering" V 7330 3350 50  0001 C CNN
 F 3 "" H 7400 3350 50  0001 C CNN
 	1    7400 3350
@@
 F 0 "R15" V 10030 3850 50  0000 C CNN
 F 1 "10k" V 9950 3850 50  0000 C CNN
-F 2 "" V 9880 3850 50  0001 C CNN
+F 2 "Resistors_SMD:R_0603_HandSoldering" V 9880 3850 50  0001 C CNN
 F 3 "" H 9950 3850 50  0001 C CNN
 	1    9950 3850
@@
 F 0 "C45" H 7410 4120 50  0000 L CNN
 F 1 "0.01uF" H 7410 3970 50  0000 L CNN
-F 2 "" H 7400 4050 50  0001 C CNN
+F 2 "Capacitors_SMD:C_0603_HandSoldering" H 7400 4050 50  0001 C CNN
 F 3 "" H 7400 4050 50  0001 C CNN
 	1    7400 4050
@@
 F 0 "JP1" H 7150 4350 50  0000 C CNN
 F 1 "Write Protect" H 7150 4120 50  0000 C CNN
-F 2 "" H 7150 4200 50  0001 C CNN
+F 2 "Capacitors_SMD:C_0603_HandSoldering" H 7150 4200 50  0001 C CNN
 F 3 "" H 7150 4200 50  0001 C CNN
 	1    7150 4200
@@
 F 0 "C46" H 10260 3770 50  0000 L CNN
 F 1 "0.01uF" H 10260 3620 50  0000 L CNN
-F 2 "" H 10250 3700 50  0001 C CNN
+F 2 "Capacitors_SMD:C_0603_HandSoldering" H 10250 3700 50  0001 C CNN
 F 3 "" H 10250 3700 50  0001 C CNN
 	1    10250 3700
@@
 F 0 "J22" H 10000 3270 50  0000 C CNN
 F 1 "TEST_1P" H 10000 3200 50  0000 C CNN
-F 2 "" H 10200 3000 50  0001 C CNN
+F 2 "SMD_Packages:1Pin" H 10200 3000 50  0001 C CNN
 F 3 "" H 10200 3000 50  0001 C CNN
 	1    10000 3000
@@
 F 0 "RN6" V 6350 5250 50  0000 C CNN
 F 1 "EXBN8V-22" V 6850 5250 50  0000 C CNN
-F 2 "" V 6925 5250 50  0001 C CNN
+F 2 "Zeabus:CRA06S" V 6925 5250 50  0001 C CNN
 F 3 "" H 6650 5250 50  0001 C CNN
 	1    6650 5250
@@
 F 0 "RN7" V 6350 5850 50  0000 C CNN
 F 1 "EXBN8V-22" V 6850 5850 50  0000 C CNN
-F 2 "" V 6925 5850 50  0001 C CNN
+F 2 "Zeabus:CRA06S" V 6925 5850 50  0001 C CNN
 F 3 "" H 6650 5850 50  0001 C CNN
 	1    6650 5850
@@
 F 0 "RN8" V 7300 5250 50  0000 C CNN
 F 1 "EXBN8V-22" V 7800 5250 50  0000 C CNN
-F 2 "" V 7875 5250 50  0001 C CNN
+F 2 "Zeabus:CRA06S" V 7875 5250 50  0001 C CNN
 F 3 "" H 7600 5250 50  0001 C CNN
 	1    7600 5250
@@
 F 0 "RN11" V 8250 5850 50  0000 C CNN
 F 1 "EXBN8V-22" V 8750 5850 50  0000 C CNN
-F 2 "" V 8825 5850 50  0001 C CNN
+F 2 "Zeabus:CRA06S" V 8825 5850 50  0001 C CNN
 F 3 "" H 8550 5850 50  0001 C CNN
 	1    8550 5850
@@
 F 0 "RN12" V 9200 5250 50  0000 C CNN
 F 1 "EXBN8V-22" V 9700 5250 50  0000 C CNN
-F 2 "" V 9775 5250 50  0001 C CNN
+F 2 "Zeabus:CRA06S" V 9775 5250 50  0001 C CNN
 F 3 "" H 9500 5250 50  0001 C CNN
 	1    9500 5250
@@
 F 0 "RN9" V 7300 5850 50  0000 C CNN
 F 1 "EXBN8V-22" V 7800 5850 50  0000 C CNN
-F 2 "" V 7875 5850 50  0001 C CNN
+F 2 "Zeabus:CRA06S" V 7875 5850 50  0001 C CNN
 F 3 "" H 7600 5850 50  0001 C CNN
 	1    7600 5850
@@
 F 0 "RN10" V 8250 5250 50  0000 C CNN
 F 1 "EXBN8V-22" V 8750 5250 50  0000 C CNN
-F 2 "" V 8825 5250 50  0001 C CNN
+F 2 "Zeabus:CRA06S" V 8825 5250 50  0001 C CNN
 F 3 "" H 8550 5250 50  0001 C CNN
 	1    8550 5250
@@
 F 0 "RN13" V 9200 5850 50  0000 C CNN
 F 1 "EXBN8V-22" V 9700 5850 50  0000 C CNN
-F 2 "" V 9775 5850 50  0001 C CNN
+F 2 "Zeabus:CRA06S" V 9775 5850 50  0001 C CNN
 F 3 "" H 9500 5850 50  0001 C CNN
 	1    9500 5850
@@
 F 0 "R10" V 10630 5350 50  0000 C CNN
 F 1 "22" V 10550 5350 50  0000 C CNN
-F 2 "" V 10480 5350 50  0001 C CNN
+F 2 "Resistors_SMD:R_0603_HandSoldering" V 10480 5350 50  0001 C CNN
 F 3 "" H 10550 5350 50  0001 C CNN
 	1    10550 5350
@@
 F 0 "R11" V 10630 5550 50  0000 C CNN
 F 1 "22" V 10550 5550 50  0000 C CNN
-F 2 "" V 10480 5550 50  0001 C CNN
+F 2 "Resistors_SMD:R_0603_HandSoldering" V 10480 5550 50  0001 C CNN
 F 3 "" H 10550 5550 50  0001 C CNN
 	1    10550 5550
@@
 F 0 "R12" V 10630 5750 50  0000 C CNN
 F 1 "22" V 10550 5750 50  0000 C CNN
-F 2 "" V 10480 5750 50  0001 C CNN
+F 2 "Resistors_SMD:R_0603_HandSoldering" V 10480 5750 50  0001 C CNN
 F 3 "" H 10550 5750 50  0001 C CNN
 	1    10550 5750
@@
 F 0 "Y1" V 3250 3650 50  0000 C CNN
 F 1 "CSTCC2M00G53-R0" V 3350 3700 50  0000 C CNN
-F 2 "" H 3575 3750 50  0001 C CNN
+F 2 "Crystals:Resonator_7.2x3mm" H 3575 3750 50  0001 C CNN
 F 3 "" H 3575 3750 50  0001 C CNN
 	1    3600 3750
@@
 F 0 "U6" H 1650 6600 45  0000 L BNN
 F 1 "ADM708SARZ" H 1600 5350 45  0000 L BNN
-F 2 "" H 1330 6500 20  0001 C CNN
+F 2 "Zeabus:ADM708_R_8" H 1330 6500 20  0001 C CNN
 F 3 "" H 1300 6350 60  0001 C CNN
 	1    1300 6350
@@
 F 0 "U4" H 2300 5150 50  0000 C CNN
 F 1 "74LVC1G08" H 2300 5050 50  0000 C CNN
-F 2 "" H 2300 5100 50  0001 C CNN
+F 2 "TO_SOT_Packages_SMD:SOT-353" H 2300 5100 50  0001 C CNN
 F 3 "" H 2300 5100 50  0001 C CNN
 	1    2300 5100
@@
 F 0 "U5" H 3600 5050 50  0000 C CNN
 F 1 "74LVC1G08" H 3600 4950 50  0000 C CNN
-F 2 "" H 3600 5000 50  0001 C CNN
+F 2 "TO_SOT_Packages_SMD:SOT-353" H 3600 5000 50  0001 C CNN
 F 3 "" H 3600 5000 50  0001 C CNN
 	1    3600 5000
@@
 F 0 "R16" V 1480 4450 50  0000 C CNN
 F 1 "10k" V 1400 4450 50  0000 C CNN
-F 2 "" V 1330 4450 50  0001 C CNN
+F 2 "Resistors_SMD:R_0603_HandSoldering" V 1330 4450 50  0001 C CNN
 F 3 "" H 1400 4450 50  0001 C CNN
 	1    1400 4450
@@
 F 0 "R17" V 1680 4450 50  0000 C CNN
 F 1 "10k" V 1600 4450 50  0000 C CNN
-F 2 "" V 1530 4450 50  0001 C CNN
+F 2 "Resistors_SMD:R_0603_HandSoldering" V 1530 4450 50  0001 C CNN
 F 3 "" H 1600 4450 50  0001 C CNN
 	1    1600 4450
@@
 F 0 "R18" V 3080 4450 50  0000 C CNN
 F 1 "10k" V 3000 4450 50  0000 C CNN
-F 2 "" V 2930 4450 50  0001 C CNN
+F 2 "Resistors_SMD:R_0603_HandSoldering" V 2930 4450 50  0001 C CNN
 F 3 "" H 3000 4450 50  0001 C CNN
 	1    3000 4450
@@
 F 0 "R19" V 4680 6300 50  0000 C CNN
 F 1 "330" V 4600 6300 50  0000 C CNN
-F 2 "" V 4530 6300 50  0001 C CNN
+F 2 "Resistors_SMD:R_0603_HandSoldering" V 4530 6300 50  0001 C CNN
 F 3 "" H 4600 6300 50  0001 C CNN
 	1    4600 6300
@@
 F 0 "D1" H 4550 6175 50  0000 L CNN
 F 1 "Yellow" V 4600 5750 50  0000 L CNN
-F 2 "" V 4600 6050 50  0001 C CNN
+F 2 "LEDs:LED_0603" V 4600 6050 50  0001 C CNN
 F 3 "" V 4600 6050 50  0001 C CNN
 	1    4600 6050
@@
 P 1200 5550
 F 0 "SW2" H 1250 5650 50  0000 L CNN
-F 1 "SW_Push_Dual" H 1200 5280 50  0000 C CNN
-F 2 "" H 1200 5750 50  0001 C CNN
+F 1 "PB" H 1200 5280 50  0000 C CNN
+F 2 "Zeabus:Button-EVQ" H 1200 5750 50  0001 C CNN
 F 3 "" H 1200 5750 50  0001 C CNN
 	1    1200 5550
@@
 F 0 "JP2" H 850 5650 50  0000 C CNN
 F 1 "External Reset" H 850 5420 50  0000 C CNN
-F 2 "" H 850 5500 50  0001 C CNN
+F 2 "Pin_Headers:Pin_Header_Straight_1x02_Pitch2.54mm" H 850 5500 50  0001 C CNN
 F 3 "" H 850 5500 50  0001 C CNN
 	1    850  5500
@@
 F 0 "C47" H 1210 7270 50  0000 L CNN
 F 1 "0.01uF" H 1210 7120 50  0000 L CNN
-F 2 "" H 1200 7200 50  0001 C CNN
+F 2 "Capacitors_SMD:C_0603_HandSoldering" H 1200 7200 50  0001 C CNN
 F 3 "" H 1200 7200 50  0001 C CNN
 	1    1200 7200

Commit message: - Add C150 - C153 at LNA input - Change value of C112, C115, C118, C221 at LNA input - Finished PCB lay-out. Ready to route
Parts:
- C45, C46, C47: footprint Capacitors_SMD:C_0603_HandSoldering -> Capacitors_SMD:C_0603
- J22: footprint SMD_Packages:1Pin -> Zeabus:1Pin-TP
- R10, R11, R12, R13, R14, R15, R16, R17, R18, R19: footprint Resistors_SMD:R_0603_HandSoldering -> Resistors_SMD:R_0603
Changed lines of the file:
@@
 F 0 "R14" V 7680 3350 50  0000 C CNN
 F 1 "10k" V 7600 3350 50  0000 C CNN
-F 2 "Resistors_SMD:R_0603_HandSoldering" V 7530 3350 50  0001 C CNN
+F 2 "Resistors_SMD:R_0603" V 7530 3350 50  0001 C CNN
 F 3 "" H 7600 3350 50  0001 C CNN
 	1    7600 3350
@@
 F 0 "R13" V 7480 3350 50  0000 C CNN
 F 1 "10k" V 7400 3350 50  0000 C CNN
-F 2 "Resistors_SMD:R_0603_HandSoldering" V 7330 3350 50  0001 C CNN
+F 2 "Resistors_SMD:R_0603" V 7330 3350 50  0001 C CNN
 F 3 "" H 7400 3350 50  0001 C CNN
 	1    7400 3350
@@
 F 0 "R15" V 10030 3850 50  0000 C CNN
 F 1 "10k" V 9950 3850 50  0000 C CNN
-F 2 "Resistors_SMD:R_0603_HandSoldering" V 9880 3850 50  0001 C CNN
+F 2 "Resistors_SMD:R_0603" V 9880 3850 50  0001 C CNN
 F 3 "" H 9950 3850 50  0001 C CNN
 	1    9950 3850
@@
 F 0 "C45" H 7410 4120 50  0000 L CNN
 F 1 "0.01uF" H 7410 3970 50  0000 L CNN
-F 2 "Capacitors_SMD:C_0603_HandSoldering" H 7400 4050 50  0001 C CNN
+F 2 "Capacitors_SMD:C_0603" H 7400 4050 50  0001 C CNN
 F 3 "" H 7400 4050 50  0001 C CNN
 	1    7400 4050
@@
 F 0 "C46" H 10260 3770 50  0000 L CNN
 F 1 "0.01uF" H 10260 3620 50  0000 L CNN
-F 2 "Capacitors_SMD:C_0603_HandSoldering" H 10250 3700 50  0001 C CNN
+F 2 "Capacitors_SMD:C_0603" H 10250 3700 50  0001 C CNN
 F 3 "" H 10250 3700 50  0001 C CNN
 	1    10250 3700
@@
 F 0 "J22" H 10000 3270 50  0000 C CNN
 F 1 "TEST_1P" H 10000 3200 50  0000 C CNN
-F 2 "SMD_Packages:1Pin" H 10200 3000 50  0001 C CNN
+F 2 "Zeabus:1Pin-TP" H 10200 3000 50  0001 C CNN
 F 3 "" H 10200 3000 50  0001 C CNN
 	1    10000 3000
@@
 F 0 "R10" V 10630 5350 50  0000 C CNN
 F 1 "22" V 10550 5350 50  0000 C CNN
-F 2 "Resistors_SMD:R_0603_HandSoldering" V 10480 5350 50  0001 C CNN
+F 2 "Resistors_SMD:R_0603" V 10480 5350 50  0001 C CNN
 F 3 "" H 10550 5350 50  0001 C CNN
 	1    10550 5350
@@
 F 0 "R11" V 10630 5550 50  0000 C CNN
 F 1 "22" V 10550 5550 50  0000 C CNN
-F 2 "Resistors_SMD:R_0603_HandSoldering" V 10480 5550 50  0001 C CNN
+F 2 "Resistors_SMD:R_0603" V 10480 5550 50  0001 C CNN
 F 3 "" H 10550 5550 50  0001 C CNN
 	1    10550 5550
@@
 F 0 "R12" V 10630 5750 50  0000 C CNN
 F 1 "22" V 10550 5750 50  0000 C CNN
-F 2 "Resistors_SMD:R_0603_HandSoldering" V 10480 5750 50  0001 C CNN
+F 2 "Resistors_SMD:R_0603" V 10480 5750 50  0001 C CNN
 F 3 "" H 10550 5750 50  0001 C CNN
 	1    10550 5750
@@
 F 0 "R16" V 1480 4450 50  0000 C CNN
 F 1 "10k" V 1400 4450 50  0000 C CNN
-F 2 "Resistors_SMD:R_0603_HandSoldering" V 1330 4450 50  0001 C CNN
+F 2 "Resistors_SMD:R_0603" V 1330 4450 50  0001 C CNN
 F 3 "" H 1400 4450 50  0001 C CNN
 	1    1400 4450
@@
 F 0 "R17" V 1680 4450 50  0000 C CNN
 F 1 "10k" V 1600 4450 50  0000 C CNN
-F 2 "Resistors_SMD:R_0603_HandSoldering" V 1530 4450 50  0001 C CNN
+F 2 "Resistors_SMD:R_0603" V 1530 4450 50  0001 C CNN
 F 3 "" H 1600 4450 50  0001 C CNN
 	1    1600 4450
@@
 F 0 "R18" V 3080 4450 50  0000 C CNN
 F 1 "10k" V 3000 4450 50  0000 C CNN
-F 2 "Resistors_SMD:R_0603_HandSoldering" V 2930 4450 50  0001 C CNN
+F 2 "Resistors_SMD:R_0603" V 2930 4450 50  0001 C CNN
 F 3 "" H 3000 4450 50  0001 C CNN
 	1    3000 4450
@@
 F 0 "R19" V 4680 6300 50  0000 C CNN
 F 1 "330" V 4600 6300 50  0000 C CNN
-F 2 "Resistors_SMD:R_0603_HandSoldering" V 4530 6300 50  0001 C CNN
+F 2 "Resistors_SMD:R_0603" V 4530 6300 50  0001 C CNN
 F 3 "" H 4600 6300 50  0001 C CNN
 	1    4600 6300
@@
 F 0 "C47" H 1210 7270 50  0000 L CNN
 F 1 "0.01uF" H 1210 7120 50  0000 L CNN
-F 2 "Capacitors_SMD:C_0603_HandSoldering" H 1200 7200 50  0001 C CNN
+F 2 "Capacitors_SMD:C_0603" H 1200 7200 50  0001 C CNN
 F 3 "" H 1200 7200 50  0001 C CNN
 	1    1200 7200
