File: DSP_Misc.sch (KiCad schematic (older format))
At the start: 46 parts, among them J18 TEST, J2 USB_OTG, J3 TEST, J4 TEST, SW3 PB0, SW4 PB0, SW5 PB0, SW6 PB0, U10 FT232RQ, U7 74LVC14, U8 74AC11244, U9 NCP361SNT1G

Commit message: First schematic release
Parts:
- C48, C49, C50, C51, C52, C53, C54, C55, C56, C57: footprint (none) -> Capacitors_SMD:C_0603_HandSoldering
- D2, D3, D4, D5, D6, D7, D8, D9: footprint (none) -> LEDs:LED_0603
- J18, J3, J4: value TEST -> TEST_1P; footprint (none) -> SMD_Packages:1Pin
- J2: footprint (none) -> Connectors:USB_Mini-B
- R20, R21, R22, R23, R24, R25, R26, R27, R28, R29, R30, R31, R32, R33, R34, R35: footprint (none) -> Resistors_SMD:R_0603_HandSoldering
- SW3, SW4, SW5, SW6: value PB0 -> PB; footprint (none) -> Zeabus:Button-EVQ
- U10: footprint (none) -> Housings_DFN_QFN:QFN-32-1EP_5x5mm_Pitch0.5mm
- U7: footprint (none) -> Housings_SSOP:SSOP-14_5.3x6.2mm_Pitch0.65mm
- U8: footprint (none) -> Housings_SSOP:TSSOP-24_4.4x7.8mm_Pitch0.65mm
- U9: footprint (none) -> Zeabus:TSOP-5

Commit message: - Add C150 - C153 at LNA input - Change value of C112, C115, C118, C221 at LNA input - Finished PCB lay-out. Ready to route
Parts:
- C48, C49, C50, C51, C52, C53, C54, C55, C56, C57: footprint Capacitors_SMD:C_0603_HandSoldering -> Capacitors_SMD:C_0603
- J18, J3, J4: footprint SMD_Packages:1Pin -> Zeabus:1Pin-TP
- R20, R21, R22, R23, R24, R25, R26, R27, R28, R29, R30, R31, R32, R33, R34, R35: footprint Resistors_SMD:R_0603_HandSoldering -> Resistors_SMD:R_0603
Changed lines of the file:
@@
 F 0 "C48" H 3010 1170 50  0000 L CNN
 F 1 "0.01uF" H 3010 1020 50  0000 L CNN
-F 2 "Capacitors_SMD:C_0603_HandSoldering" H 3000 1100 50  0001 C CNN
+F 2 "Capacitors_SMD:C_0603" H 3000 1100 50  0001 C CNN
 F 3 "" H 3000 1100 50  0001 C CNN
 	1    3000 1100
@@
 F 0 "R21" V 2530 1250 50  0000 C CNN
 F 1 "10k" V 2450 1250 50  0000 C CNN
-F 2 "Resistors_SMD:R_0603_HandSoldering" V 2380 1250 50  0001 C CNN
+F 2 "Resistors_SMD:R_0603" V 2380 1250 50  0001 C CNN
 F 3 "" H 2450 1250 50  0001 C CNN
 	1    2450 1250
@@
 F 0 "R20" V 2080 1500 50  0000 C CNN
 F 1 "100" V 2000 1500 50  0000 C CNN
-F 2 "Resistors_SMD:R_0603_HandSoldering" V 1930 1500 50  0001 C CNN
+F 2 "Resistors_SMD:R_0603" V 1930 1500 50  0001 C CNN
 F 3 "" H 2000 1500 50  0001 C CNN
 	1    2000 1500
@@
 F 0 "C49" H 2460 1820 50  0000 L CNN
 F 1 "1uF" H 2460 1670 50  0000 L CNN
-F 2 "Capacitors_SMD:C_0603_HandSoldering" H 2450 1750 50  0001 C CNN
+F 2 "Capacitors_SMD:C_0603" H 2450 1750 50  0001 C CNN
 F 3 "" H 2450 1750 50  0001 C CNN
 	1    2450 1750
@@
 F 0 "R29" V 8080 2100 50  0000 C CNN
 F 1 "330" V 8000 2100 50  0000 C CNN
-F 2 "Resistors_SMD:R_0603_HandSoldering" V 7930 2100 50  0001 C CNN
+F 2 "Resistors_SMD:R_0603" V 7930 2100 50  0001 C CNN
 F 3 "" H 8000 2100 50  0001 C CNN
 	1    8000 2100
@@
 F 0 "R23" V 2530 2400 50  0000 C CNN
 F 1 "10k" V 2450 2400 50  0000 C CNN
-F 2 "Resistors_SMD:R_0603_HandSoldering" V 2380 2400 50  0001 C CNN
+F 2 "Resistors_SMD:R_0603" V 2380 2400 50  0001 C CNN
 F 3 "" H 2450 2400 50  0001 C CNN
 	1    2450 2400
@@
 F 0 "R22" V 2080 2650 50  0000 C CNN
 F 1 "100" V 2000 2650 50  0000 C CNN
-F 2 "Resistors_SMD:R_0603_HandSoldering" V 1930 2650 50  0001 C CNN
+F 2 "Resistors_SMD:R_0603" V 1930 2650 50  0001 C CNN
 F 3 "" H 2000 2650 50  0001 C CNN
 	1    2000 2650
@@
 F 0 "C50" H 2460 2970 50  0000 L CNN
 F 1 "1uF" H 2460 2820 50  0000 L CNN
-F 2 "Capacitors_SMD:C_0603_HandSoldering" H 2450 2900 50  0001 C CNN
+F 2 "Capacitors_SMD:C_0603" H 2450 2900 50  0001 C CNN
 F 3 "" H 2450 2900 50  0001 C CNN
 	1    2450 2900
@@
 F 0 "R25" V 2530 3600 50  0000 C CNN
 F 1 "10k" V 2450 3600 50  0000 C CNN
-F 2 "Resistors_SMD:R_0603_HandSoldering" V 2380 3600 50  0001 C CNN
+F 2 "Resistors_SMD:R_0603" V 2380 3600 50  0001 C CNN
 F 3 "" H 2450 3600 50  0001 C CNN
 	1    2450 3600
@@
 F 0 "R24" V 2080 3850 50  0000 C CNN
 F 1 "100" V 2000 3850 50  0000 C CNN
-F 2 "Resistors_SMD:R_0603_HandSoldering" V 1930 3850 50  0001 C CNN
+F 2 "Resistors_SMD:R_0603" V 1930 3850 50  0001 C CNN
 F 3 "" H 2000 3850 50  0001 C CNN
 	1    2000 3850
@@
 F 0 "C51" H 2460 4170 50  0000 L CNN
 F 1 "1uF" H 2460 4020 50  0000 L CNN
-F 2 "Capacitors_SMD:C_0603_HandSoldering" H 2450 4100 50  0001 C CNN
+F 2 "Capacitors_SMD:C_0603" H 2450 4100 50  0001 C CNN
 F 3 "" H 2450 4100 50  0001 C CNN
 	1    2450 4100
@@
 F 0 "R27" V 2530 4800 50  0000 C CNN
 F 1 "10k" V 2450 4800 50  0000 C CNN
-F 2 "Resistors_SMD:R_0603_HandSoldering" V 2380 4800 50  0001 C CNN
+F 2 "Resistors_SMD:R_0603" V 2380 4800 50  0001 C CNN
 F 3 "" H 2450 4800 50  0001 C CNN
 	1    2450 4800
@@
 F 0 "R26" V 2080 5050 50  0000 C CNN
 F 1 "100" V 2000 5050 50  0000 C CNN
-F 2 "Resistors_SMD:R_0603_HandSoldering" V 1930 5050 50  0001 C CNN
+F 2 "Resistors_SMD:R_0603" V 1930 5050 50  0001 C CNN
 F 3 "" H 2000 5050 50  0001 C CNN
 	1    2000 5050
@@
 F 0 "C52" H 2460 5370 50  0000 L CNN
 F 1 "1uF" H 2460 5220 50  0000 L CNN
-F 2 "Capacitors_SMD:C_0603_HandSoldering" H 2450 5300 50  0001 C CNN
+F 2 "Capacitors_SMD:C_0603" H 2450 5300 50  0001 C CNN
 F 3 "" H 2450 5300 50  0001 C CNN
 	1    2450 5300
@@
 F 0 "C53" H 7460 2420 50  0000 L CNN
 F 1 "0.01uF" H 7460 2270 50  0000 L CNN
-F 2 "Capacitors_SMD:C_0603_HandSoldering" H 7450 2350 50  0001 C CNN
+F 2 "Capacitors_SMD:C_0603" H 7450 2350 50  0001 C CNN
 F 3 "" H 7450 2350 50  0001 C CNN
 	1    7450 2350
@@
 F 0 "R30" V 8430 2100 50  0000 C CNN
 F 1 "330" V 8350 2100 50  0000 C CNN
-F 2 "Resistors_SMD:R_0603_HandSoldering" V 8280 2100 50  0001 C CNN
+F 2 "Resistors_SMD:R_0603" V 8280 2100 50  0001 C CNN
 F 3 "" H 8350 2100 50  0001 C CNN
 	1    8350 2100
@@
 F 0 "R31" V 8780 2100 50  0000 C CNN
 F 1 "330" V 8700 2100 50  0000 C CNN
-F 2 "Resistors_SMD:R_0603_HandSoldering" V 8630 2100 50  0001 C CNN
+F 2 "Resistors_SMD:R_0603" V 8630 2100 50  0001 C CNN
 F 3 "" H 8700 2100 50  0001 C CNN
 	1    8700 2100
@@
 F 0 "R32" V 9130 2100 50  0000 C CNN
 F 1 "330" V 9050 2100 50  0000 C CNN
-F 2 "Resistors_SMD:R_0603_HandSoldering" V 8980 2100 50  0001 C CNN
+F 2 "Resistors_SMD:R_0603" V 8980 2100 50  0001 C CNN
 F 3 "" H 9050 2100 50  0001 C CNN
 	1    9050 2100
@@
 F 0 "R28" V 1630 6000 50  0000 C CNN
 F 1 "10k" V 1550 6000 50  0000 C CNN
-F 2 "Resistors_SMD:R_0603_HandSoldering" V 1480 6000 50  0001 C CNN
+F 2 "Resistors_SMD:R_0603" V 1480 6000 50  0001 C CNN
 F 3 "" H 1550 6000 50  0001 C CNN
 	1    1550 6000
@@
 F 0 "C55" H 5510 3870 50  0000 L CNN
 F 1 "0.01uF" H 5510 3720 50  0000 L CNN
-F 2 "Capacitors_SMD:C_0603_HandSoldering" H 5500 3800 50  0001 C CNN
+F 2 "Capacitors_SMD:C_0603" H 5500 3800 50  0001 C CNN
 F 3 "" H 5500 3800 50  0001 C CNN
 	1    5500 3800
@@
 F 0 "C54" H 5260 3870 50  0000 L CNN
 F 1 "1uF" H 5260 3720 50  0000 L CNN
-F 2 "Capacitors_SMD:C_0603_HandSoldering" H 5250 3800 50  0001 C CNN
+F 2 "Capacitors_SMD:C_0603" H 5250 3800 50  0001 C CNN
 F 3 "" H 5250 3800 50  0001 C CNN
 	1    5250 3800
@@
 F 0 "J18" H 5900 4270 50  0000 C CNN
 F 1 "TEST_1P" V 5800 4050 50  0000 C CNN
-F 2 "SMD_Packages:1Pin" H 6100 4000 50  0001 C CNN
+F 2 "Zeabus:1Pin-TP" H 6100 4000 50  0001 C CNN
 F 3 "" H 6100 4000 50  0001 C CNN
 	1    5900 4000
@@
 F 0 "J3" H 7750 6020 50  0000 C CNN
 F 1 "TEST_1P" H 7750 5950 50  0000 C CNN
-F 2 "SMD_Packages:1Pin" H 7950 5750 50  0001 C CNN
+F 2 "Zeabus:1Pin-TP" H 7950 5750 50  0001 C CNN
 F 3 "" H 7950 5750 50  0001 C CNN
 	1    7750 5750
@@
 F 0 "C57" H 7460 4420 50  0000 L CNN
 F 1 "0.1uF" H 7460 4270 50  0000 L CNN
-F 2 "Capacitors_SMD:C_0603_HandSoldering" H 7450 4350 50  0001 C CNN
+F 2 "Capacitors_SMD:C_0603" H 7450 4350 50  0001 C CNN
 F 3 "" H 7450 4350 50  0001 C CNN
 	1    7450 4350
@@
 F 0 "C56" H 7410 3870 50  0000 L CNN
 F 1 "1uF" H 7410 3720 50  0000 L CNN
-F 2 "Capacitors_SMD:C_0603_HandSoldering" H 7400 3800 50  0001 C CNN
+F 2 "Capacitors_SMD:C_0603" H 7400 3800 50  0001 C CNN
 F 3 "" H 7400 3800 50  0001 C CNN
 	1    7400 3800
@@
 F 0 "R33" V 9830 5200 50  0000 C CNN
 F 1 "330" V 9750 5200 50  0000 C CNN
-F 2 "Resistors_SMD:R_0603_HandSoldering" V 9680 5200 50  0001 C CNN
+F 2 "Resistors_SMD:R_0603" V 9680 5200 50  0001 C CNN
 F 3 "" H 9750 5200 50  0001 C CNN
 	1    9750 5200
@@
 F 0 "R34" V 10180 5200 50  0000 C CNN
 F 1 "330" V 10100 5200 50  0000 C CNN
-F 2 "Resistors_SMD:R_0603_HandSoldering" V 10030 5200 50  0001 C CNN
+F 2 "Resistors_SMD:R_0603" V 10030 5200 50  0001 C CNN
 F 3 "" H 10100 5200 50  0001 C CNN
 	1    10100 5200
@@
 F 0 "R35" V 10530 5200 50  0000 C CNN
 F 1 "330" V 10450 5200 50  0000 C CNN
-F 2 "Resistors_SMD:R_0603_HandSoldering" V 10380 5200 50  0001 C CNN
+F 2 "Resistors_SMD:R_0603" V 10380 5200 50  0001 C CNN
 F 3 "" H 10450 5200 50  0001 C CNN
 	1    10450 5200
@@
 F 0 "J4" H 9350 5920 50  0000 C CNN
 F 1 "TEST_1P" V 9450 5900 50  0000 C CNN
-F 2 "SMD_Packages:1Pin" H 9550 5650 50  0001 C CNN
+F 2 "Zeabus:1Pin-TP" H 9550 5650 50  0001 C CNN
 F 3 "" H 9550 5650 50  0001 C CNN
 	1    9350 5650
@@
 	1    0    0    -1
 $EndComp
+Connection ~ 5500 4200
 $EndSCHEMATC
