File: LNA.sch (KiCad schematic (older format))
At the start: 77 parts, among them CN1 EPS.00.250.NTN, CN2 EPS.00.250.NTN, CN3 EPS.00.250.NTN, CN4 EPS.00.250.NTN, J14 TEST_1P, J15 TEST_1P, J16 TEST_1P, J17 TEST_1P, U18 AD8334ACPZ

Commit message: First schematic release
Parts:
- C112, C113, C114, C115, C116, C117, C118, C119, C120, C121, C122, C123, C124, C125, C126, C127, C128, C129, C130, C131, C132, C133, C134, C135, C136, C137, C138, C139, C140, C141, C142, C143, C144, C145: footprint (none) -> Capacitors_SMD:C_0603_HandSoldering
- J14, J15, J16, J17: footprint (none) -> SMD_Packages:1Pin
- L1, L3, L5, L7: footprint (none) -> Zeabus:L-SDR0503
- L10, L11, L12, L13, L14, L15, L16, L17, L18, L19, L2, L20, L21, L22, L4, L6, L8, L9: footprint (none) -> Inductors_SMD:L_0603_HandSoldering
- R79, R80, R81, R82, R83, R84, R85, R86, R87, R88, R89, R90: footprint (none) -> Resistors_SMD:R_0603_HandSoldering
- U18: footprint (none) -> Zeabus:QFN50P900X900X100-65N
Connections:
- net labels added: IN1, IN2, IN3, IN4

Commit message: - Add C150 - C153 at LNA input - Change value of C112, C115, C118, C221 at LNA input - Finished PCB lay-out. Ready to route
Parts:
- added C150, C151, C152, C153: 0.1uF, Capacitors_SMD:C_0603, symbol C_Small
- C112, C115, C118, C121: value 0.1uF -> 22pF; footprint Capacitors_SMD:C_0603_HandSoldering -> Capacitors_SMD:C_0603
- C113, C114, C116, C117, C119, C120, C122, C123, C124, C125, C126, C127, C128, C129, C130, C131, C132, C133, C134, C135, C136, C137, C138, C139, C140, C141, C142, C143, C144, C145: footprint Capacitors_SMD:C_0603_HandSoldering -> Capacitors_SMD:C_0603
- J14, J15, J16, J17: footprint SMD_Packages:1Pin -> Zeabus:1Pin-TP
- L10, L11, L12, L13, L14, L15, L16, L17, L18, L19, L2, L20, L21, L22, L4, L6, L8, L9: footprint Inductors_SMD:L_0603_HandSoldering -> Inductors_SMD:L_0603
- R79, R80, R81, R82, R83, R84, R85, R86, R87, R88, R89, R90: footprint Resistors_SMD:R_0603_HandSoldering -> Resistors_SMD:R_0603
Connections:
- wire segments 225 -> 229
