File: LNA_Gain_Ctrl.sch (KiCad schematic (older format))
At the start: 8 parts, among them U19 MAX5387LAUD+T, U20 TLV3311P

Commit message: First schematic release
Parts:
- added R100, R99: 10k, Resistors_SMD:R_0603_HandSoldering, symbol R
- R93, R94, R95, R96, R97, R98: footprint (none) -> Resistors_SMD:R_0603_HandSoldering
- U19: footprint (none) -> Housings_SSOP:TSSOP-14_4.4x5mm_Pitch0.65mm
- U20: value TLV3311P -> TLV73311PDBVT; footprint (none) -> TO_SOT_Packages_SMD:SOT-23-5_HandSoldering; symbol TLV33 -> TLV733
Changed lines of the file:
@@
 LIBS:zeabus
 LIBS:ftdi
+LIBS:Zeabus-Elec-Hydrophone-cache
 EELAYER 25 0
 EELAYER END
@@
 F 0 "U19" H 5668 4462 45  0000 L BNN
 F 1 "MAX5387LAUD+T" H 5567 2801 45  0000 L BNN
-F 2 "" H 5880 3900 20  0001 C CNN
+F 2 "Housings_SSOP:TSSOP-14_4.4x5mm_Pitch0.65mm" H 5880 3900 20  0001 C CNN
 F 3 "" H 5850 3750 60  0001 C CNN
 	1    5850 3750
@@
 $EndComp
 $Comp
-L GNDA #PWR0137
+L GNDA #PWR0138
 U 1 1 599B078D
 P 7350 2300
-F 0 "#PWR0137" H 7350 2050 50  0001 C CNN
+F 0 "#PWR0138" H 7350 2050 50  0001 C CNN
 F 1 "GNDA" H 7350 2150 50  0000 C CNN
 F 2 "" H 7350 2300 50  0001 C CNN
@@
 $EndComp
 $Comp
-L +3.3VA #PWR0138
+L +3.3VA #PWR0139
 U 1 1 599B07B0
 P 8250 2050
-F 0 "#PWR0138" H 8250 1900 50  0001 C CNN
+F 0 "#PWR0139" H 8250 1900 50  0001 C CNN
 F 1 "+3.3VA" H 8250 2190 50  0000 C CNN
 F 2 "" H 8250 2050 50  0001 C CNN
@@
 	6600 3950 6550 3950
 $Comp
-L GNDA #PWR0139
+L GNDA #PWR0140
 U 1 1 599B08BC
 P 7000 4050
-F 0 "#PWR0139" H 7000 3800 50  0001 C CNN
+F 0 "#PWR0140" H 7000 3800 50  0001 C CNN
 F 1 "GNDA" H 7000 3900 50  0000 C CNN
 F 2 "" H 7000 4050 50  0001 C CNN
@@
 	5150 4150 5150 4450
 $Comp
-L GNDD #PWR0140
+L GNDD #PWR0141
 U 1 1 599B08F3
 P 5150 4450
-F 0 "#PWR0140" H 5150 4200 50  0001 C CNN
+F 0 "#PWR0141" H 5150 4200 50  0001 C CNN
 F 1 "GNDD" H 5150 4300 50  0000 C CNN
 F 2 "" H 5150 4450 50  0001 C CNN
@@
 $EndComp
 $Comp
-L +3.3V #PWR0141
+L +3.3V #PWR0142
 U 1 1 599B0916
 P 5150 3150
-F 0 "#PWR0141" H 5150 3000 50  0001 C CNN
+F 0 "#PWR0142" H 5150 3000 50  0001 C CNN
 F 1 "+3.3V" H 5150 3290 50  0000 C CNN
 F 2 "" H 5150 3150 50  0001 C CNN
@@
 F 0 "R96" V 4180 4200 50  0000 C CNN
 F 1 "10k" V 4100 4200 50  0000 C CNN
-F 2 "" V 4030 4200 50  0001 C CNN
+F 2 "Resistors_SMD:R_0603_HandSoldering" V 4030 4200 50  0001 C CNN
 F 3 "" H 4100 4200 50  0001 C CNN
 	1    4100 4200
@@
 F 0 "R97" V 4380 4200 50  0000 C CNN
 F 1 "10k" V 4300 4200 50  0000 C CNN
-F 2 "" V 4230 4200 50  0001 C CNN
+F 2 "Resistors_SMD:R_0603_HandSoldering" V 4230 4200 50  0001 C CNN
 F 3 "" H 4300 4200 50  0001 C CNN
 	1    4300 4200
@@
 F 0 "R98" V 4580 4200 50  0000 C CNN
 F 1 "10k" V 4500 4200 50  0000 C CNN
-F 2 "" V 4430 4200 50  0001 C CNN
+F 2 "Resistors_SMD:R_0603_HandSoldering" V 4430 4200 50  0001 C CNN
 F 3 "" H 4500 4200 50  0001 C CNN
 	1    4500 4200
@@
 F 0 "R93" V 4180 3400 50  0000 C CNN
 F 1 "0" V 4100 3400 50  0000 C CNN
-F 2 "" V 4030 3400 50  0001 C CNN
+F 2 "Resistors_SMD:R_0603_HandSoldering" V 4030 3400 50  0001 C CNN
 F 3 "" H 4100 3400 50  0001 C CNN
 	1    4100 3400
@@
 F 0 "R94" V 4380 3400 50  0000 C CNN
 F 1 "0" V 4300 3400 50  0000 C CNN
-F 2 "" V 4230 3400 50  0001 C CNN
+F 2 "Resistors_SMD:R_0603_HandSoldering" V 4230 3400 50  0001 C CNN
 F 3 "" H 4300 3400 50  0001 C CNN
 	1    4300 3400
@@
 F 0 "R95" V 4580 3400 50  0000 C CNN
 F 1 "0" V 4500 3400 50  0000 C CNN
-F 2 "" V 4430 3400 50  0001 C CNN
+F 2 "Resistors_SMD:R_0603_HandSoldering" V 4430 3400 50  0001 C CNN
 F 3 "" H 4500 3400 50  0001 C CNN
 	1    4500 3400
@@
 	3600 3600 3600 3150
 $Comp
-L TLV33 U20
+L TLV733 U20
 U 1 1 599B876C
 P 8050 2050
 F 0 "U20" H 8150 2100 60  0000 C CNN
-F 1 "TLV3311P" H 8200 1650 60  0000 C CNN
-F 2 "" H 8050 2100 60  0001 C CNN
+F 1 "TLV73311PDBVT" H 8200 1650 60  0000 C CNN
+F 2 "TO_SOT_Packages_SMD:SOT-23-5_HandSoldering" H 8050 2100 60  0001 C CNN
 F 3 "" H 8050 2100 60  0001 C CNN
 	1    8050 2050
@@
 	8250 2050 8250 2300
 Connection ~ 8250 2150
+$Comp
+L R R99
+U 1 1 599D7AE3
+P 5050 3400
+F 0 "R99" V 5130 3400 50  0000 C CNN
+F 1 "10k" V 5050 3400 50  0000 C CNN
+F 2 "Resistors_SMD:R_0603_HandSoldering" V 4980 3400 50  0001 C CNN
+F 3 "" H 5050 3400 50  0001 C CNN
+	1    5050 3400
+	1    0    0    -1
+$EndComp
+Connection ~ 5050 3550
+Connection ~ 5050 3250
+$Comp
+L R R100
+U 1 1 599D7B87
+P 6600 3200
+F 0 "R100" V 6680 3200 50  0000 C CNN
+F 1 "10k" V 6600 3200 50  0000 C CNN
+F 2 "Resistors_SMD:R_0603_HandSoldering" V 6530 3200 50  0001 C CNN
+F 3 "" H 6600 3200 50  0001 C CNN
+	1    6600 3200
+	1    0    0    -1
+$EndComp
+Connection ~ 6600 3350
+$Comp
+L +3.3V #PWR?
+U 1 1 599D7C09
+P 6600 3050
+F 0 "#PWR?" H 6600 2900 50  0001 C CNN
+F 1 "+3.3V" H 6600 3190 50  0000 C CNN
+F 2 "" H 6600 3050 50  0001 C CNN
+F 3 "" H 6600 3050 50  0001 C CNN
+	1    6600 3050
+	1    0    0    -1
+$EndComp
 $EndSCHEMATC

Commit message: - Add C150 - C153 at LNA input - Change value of C112, C115, C118, C221 at LNA input - Finished PCB lay-out. Ready to route
Parts:
- R100, R93, R94, R95, R96, R97, R98, R99: footprint Resistors_SMD:R_0603_HandSoldering -> Resistors_SMD:R_0603
- U20: footprint TO_SOT_Packages_SMD:SOT-23-5_HandSoldering -> TO_SOT_Packages_SMD:SOT-23-5
Changed lines of the file:
@@
 F 0 "R96" V 4180 4200 50  0000 C CNN
 F 1 "10k" V 4100 4200 50  0000 C CNN
-F 2 "Resistors_SMD:R_0603_HandSoldering" V 4030 4200 50  0001 C CNN
+F 2 "Resistors_SMD:R_0603" V 4030 4200 50  0001 C CNN
 F 3 "" H 4100 4200 50  0001 C CNN
 	1    4100 4200
@@
 F 0 "R97" V 4380 4200 50  0000 C CNN
 F 1 "10k" V 4300 4200 50  0000 C CNN
-F 2 "Resistors_SMD:R_0603_HandSoldering" V 4230 4200 50  0001 C CNN
+F 2 "Resistors_SMD:R_0603" V 4230 4200 50  0001 C CNN
 F 3 "" H 4300 4200 50  0001 C CNN
 	1    4300 4200
@@
 F 0 "R98" V 4580 4200 50  0000 C CNN
 F 1 "10k" V 4500 4200 50  0000 C CNN
-F 2 "Resistors_SMD:R_0603_HandSoldering" V 4430 4200 50  0001 C CNN
+F 2 "Resistors_SMD:R_0603" V 4430 4200 50  0001 C CNN
 F 3 "" H 4500 4200 50  0001 C CNN
 	1    4500 4200
@@
 F 0 "R93" V 4180 3400 50  0000 C CNN
 F 1 "0" V 4100 3400 50  0000 C CNN
-F 2 "Resistors_SMD:R_0603_HandSoldering" V 4030 3400 50  0001 C CNN
+F 2 "Resistors_SMD:R_0603" V 4030 3400 50  0001 C CNN
 F 3 "" H 4100 3400 50  0001 C CNN
 	1    4100 3400
@@
 F 0 "R94" V 4380 3400 50  0000 C CNN
 F 1 "0" V 4300 3400 50  0000 C CNN
-F 2 "Resistors_SMD:R_0603_HandSoldering" V 4230 3400 50  0001 C CNN
+F 2 "Resistors_SMD:R_0603" V 4230 3400 50  0001 C CNN
 F 3 "" H 4300 3400 50  0001 C CNN
 	1    4300 3400
@@
 F 0 "R95" V 4580 3400 50  0000 C CNN
 F 1 "0" V 4500 3400 50  0000 C CNN
-F 2 "Resistors_SMD:R_0603_HandSoldering" V 4430 3400 50  0001 C CNN
+F 2 "Resistors_SMD:R_0603" V 4430 3400 50  0001 C CNN
 F 3 "" H 4500 3400 50  0001 C CNN
 	1    4500 3400
@@
 F 0 "U20" H 8150 2100 60  0000 C CNN
 F 1 "TLV73311PDBVT" H 8200 1650 60  0000 C CNN
-F 2 "TO_SOT_Packages_SMD:SOT-23-5_HandSoldering" H 8050 2100 60  0001 C CNN
+F 2 "TO_SOT_Packages_SMD:SOT-23-5" H 8050 2100 60  0001 C CNN
 F 3 "" H 8050 2100 60  0001 C CNN
 	1    8050 2050
@@
 F 0 "R99" V 5130 3400 50  0000 C CNN
 F 1 "10k" V 5050 3400 50  0000 C CNN
-F 2 "Resistors_SMD:R_0603_HandSoldering" V 4980 3400 50  0001 C CNN
+F 2 "Resistors_SMD:R_0603" V 4980 3400 50  0001 C CNN
 F 3 "" H 5050 3400 50  0001 C CNN
 	1    5050 3400
@@
 F 0 "R100" V 6680 3200 50  0000 C CNN
 F 1 "10k" V 6600 3200 50  0000 C CNN
-F 2 "Resistors_SMD:R_0603_HandSoldering" V 6530 3200 50  0001 C CNN
+F 2 "Resistors_SMD:R_0603" V 6530 3200 50  0001 C CNN
 F 3 "" H 6600 3200 50  0001 C CNN
 	1    6600 3200
@@
 Connection ~ 6600 3350
 $Comp
-L +3.3V #PWR?
+L +3.3V #PWR0143
 U 1 1 599D7C09
 P 6600 3050
-F 0 "#PWR?" H 6600 2900 50  0001 C CNN
+F 0 "#PWR0143" H 6600 2900 50  0001 C CNN
 F 1 "+3.3V" H 6600 3190 50  0000 C CNN
 F 2 "" H 6600 3050 50  0001 C CNN
