File: Power_Amp.sch (KiCad schematic (older format))
At the start: 104 parts, among them J10 TEST_1P, J11 TEST_1P, J12 TEST_1P, J13 TEST_1P, J6 TEST_1P, J7 TEST_1P, J8 TEST_1P, J9 TEST_1P, U14 AD8652ARZ, U15 AD8652ARZ, U16 AD8652ARZ, U17 AD8652ARZ

Commit message: First schematic release
Parts:
- C100, C101, C103, C104, C106, C108, C109, C111, C146, C64, C65, C67, C68, C70, C72, C73, C75, C76, C77, C79, C80, C82, C84, C85, C87, C88, C89, C91, C92, C94, C96, C97, C99: footprint (none) -> Capacitors_SMD:C_0603_HandSoldering
- C102, C105, C107, C110, C66, C69, C71, C74, C78, C81, C83, C86, C90, C93, C95, C98: footprint (none) -> Capacitors_SMD:C_0805_HandSoldering; symbol CP1_Small -> C_Small
- C147: footprint (none) -> Capacitors_SMD:C_0603_HandSoldering; symbol CP1_Small -> C_Small
- J10, J11, J12, J13, J6, J7, J8, J9: footprint (none) -> SMD_Packages:1Pin
- R39, R40, R41, R42, R43, R44, R45, R46, R47, R48, R49, R50, R51, R52, R53, R54, R55, R56, R57, R58, R59, R60, R61, R62, R63, R64, R65, R66, R67, R68, R69, R70, R71, R72, R73, R74, R75, R76, R77, R78, R91, R92: footprint (none) -> Resistors_SMD:R_0603_HandSoldering
- U14, U15, U16, U17: footprint (none) -> Housings_SOIC:SOIC-8_3.9x4.9mm_Pitch1.27mm

Commit message: - Add C150 - C153 at LNA input - Change value of C112, C115, C118, C221 at LNA input - Finished PCB lay-out. Ready to route
Parts:
- C100, C101, C103, C104, C106, C108, C109, C111, C146, C147, C64, C65, C67, C68, C70, C72, C73, C75, C76, C77, C79, C80, C82, C84, C85, C87, C88, C89, C91, C92, C94, C96, C97, C99: footprint Capacitors_SMD:C_0603_HandSoldering -> Capacitors_SMD:C_0603
- C102, C105, C107, C110, C66, C69, C71, C74, C78, C81, C83, C86, C90, C93, C95, C98: footprint Capacitors_SMD:C_0805_HandSoldering -> Capacitors_SMD:C_0603
- J10, J11, J12, J13, J6, J7, J8, J9: footprint SMD_Packages:1Pin -> Zeabus:1Pin-TP
- R39, R40, R41, R42, R43, R44, R45, R46, R47, R48, R49, R50, R51, R52, R53, R54, R55, R56, R57, R58, R59, R60, R61, R62, R63, R64, R65, R66, R67, R68, R69, R70, R71, R72, R73, R74, R75, R76, R77, R78, R91, R92: footprint Resistors_SMD:R_0603_HandSoldering -> Resistors_SMD:R_0603
