File: Zeabus-Elec-Hydrophone.sch (KiCad schematic (older format))
At the start: 0 parts

Commit message: First release of the schematic.
Parts:
- added C148, C149: 1uF, symbol C_Small
- added U21, U23: LM1117-3.3, symbol LM1117-3.3
- added U22: TLV3311P, symbol TLV33
Connections:
- net labels added: +1V1, +3.3V, +3.3VA, +5V, GND, GNDA, GNDD
- wire segments 0 -> 68
Other:
- note added: "Ground Junction"
- note added: "Power Supply for Analog Components"
- note added: "Power Supply for Digital Components"

Commit message: First schematic release
Parts:
- C148, C149: footprint (none) -> Capacitors_SMD:C_0603_HandSoldering
- U21, U23: footprint (none) -> TO_SOT_Packages_SMD:SOT-223-3Lead_TabPin2
- U22: value TLV3311P -> TLV73311PDVBT; footprint (none) -> TO_SOT_Packages_SMD:SOT-23-5_HandSoldering; symbol TLV33 -> TLV733
Changed lines of the file:
@@
 LIBS:zeabus
 LIBS:ftdi
+LIBS:Zeabus-Elec-Hydrophone-cache
 EELAYER 25 0
 EELAYER END
@@
 F 0 "U21" H 2550 900 50  0000 C CNN
 F 1 "LM1117-3.3" H 2450 1400 50  0000 C CNN
-F 2 "" H 2450 1150 50  0001 C CNN
+F 2 "TO_SOT_Packages_SMD:SOT-223-3Lead_TabPin2" H 2450 1150 50  0001 C CNN
 F 3 "" H 2450 1150 50  0001 C CNN
 	1    2450 1150
@@
 F 0 "U23" H 2550 2250 50  0000 C CNN
 F 1 "LM1117-3.3" H 2450 2750 50  0000 C CNN
-F 2 "" H 2450 2500 50  0001 C CNN
+F 2 "TO_SOT_Packages_SMD:SOT-223-3Lead_TabPin2" H 2450 2500 50  0001 C CNN
 F 3 "" H 2450 2500 50  0001 C CNN
 	1    2450 2500
@@
 $EndComp
 $Comp
-L TLV33 U22
+L TLV733 U22
 U 1 1 599B98B8
 P 3700 1050
 F 0 "U22" H 3800 1100 60  0000 C CNN
-F 1 "TLV3311P" H 3850 650 60  0000 C CNN
-F 2 "" H 3700 1100 60  0001 C CNN
+F 1 "TLV73311PDVBT" H 3850 650 60  0000 C CNN
+F 2 "TO_SOT_Packages_SMD:SOT-23-5_HandSoldering" H 3700 1100 60  0001 C CNN
 F 3 "" H 3700 1100 60  0001 C CNN
 	1    3700 1050
@@
 F 0 "C148" H 3110 1420 50  0000 L CNN
 F 1 "1uF" H 3110 1270 50  0000 L CNN
-F 2 "" H 3100 1350 50  0001 C CNN
+F 2 "Capacitors_SMD:C_0603_HandSoldering" H 3100 1350 50  0001 C CNN
 F 3 "" H 3100 1350 50  0001 C CNN
 	1    3100 1350
@@
 F 0 "C149" H 3060 2720 50  0000 L CNN
 F 1 "1uF" H 3060 2570 50  0000 L CNN
-F 2 "" H 3050 2650 50  0001 C CNN
+F 2 "Capacitors_SMD:C_0603_HandSoldering" H 3050 2650 50  0001 C CNN
 F 3 "" H 3050 2650 50  0001 C CNN
 	1    3050 2650

Commit message: - Add C150 - C153 at LNA input - Change value of C112, C115, C118, C221 at LNA input - Finished PCB lay-out. Ready to route
Parts:
- C148, C149: footprint Capacitors_SMD:C_0603_HandSoldering -> Capacitors_SMD:C_0603
- U22: footprint TO_SOT_Packages_SMD:SOT-23-5_HandSoldering -> TO_SOT_Packages_SMD:SOT-23-5
Changed lines of the file:
@@
 F 0 "U22" H 3800 1100 60  0000 C CNN
 F 1 "TLV73311PDVBT" H 3850 650 60  0000 C CNN
-F 2 "TO_SOT_Packages_SMD:SOT-23-5_HandSoldering" H 3700 1100 60  0001 C CNN
+F 2 "TO_SOT_Packages_SMD:SOT-23-5" H 3700 1100 60  0001 C CNN
 F 3 "" H 3700 1100 60  0001 C CNN
 	1    3700 1050
@@
 F 0 "C148" H 3110 1420 50  0000 L CNN
 F 1 "1uF" H 3110 1270 50  0000 L CNN
-F 2 "Capacitors_SMD:C_0603_HandSoldering" H 3100 1350 50  0001 C CNN
+F 2 "Capacitors_SMD:C_0603" H 3100 1350 50  0001 C CNN
 F 3 "" H 3100 1350 50  0001 C CNN
 	1    3100 1350
@@
 F 0 "C149" H 3060 2720 50  0000 L CNN
 F 1 "1uF" H 3060 2570 50  0000 L CNN
-F 2 "Capacitors_SMD:C_0603_HandSoldering" H 3050 2650 50  0001 C CNN
+F 2 "Capacitors_SMD:C_0603" H 3050 2650 50  0001 C CNN
 F 3 "" H 3050 2650 50  0001 C CNN
 	1    3050 2650
